File: PCB/hackpad actual.kicad_pcb (KiCad board)
At the start: 2 copper layers, 92.9 x 73.8 mm, 7 parts, among them SW1 SW_Push, SW2 SW_Push, SW3 SW_Push, SW4 SW_Push, SW5 SW_Push, SW6 RotaryEncoder_Switch, U1 XIAO-RP2040-DIP

Commit message: rereview edits
Routing:
- net Net-(U1-GPIO4/MISO): track 41.5 -> 93.8 mm
- net Net-(U1-GPIO6/SDA): track 88.4 -> 37.4 mm
- net Net-(U1-GPIO2/SCK): track 26.8 -> 70.5 mm
- net GND: track 167.6 -> 193.5 mm
- net Net-(U1-GPIO26/ADC0/A0): track 66.4 -> 54.3 mm
- net Net-(U1-GPIO1/RX): track 15.4 -> 19.3 mm
- net Net-(U1-GPIO3/MOSI): track 41.9 -> 44.3 mm
- net Net-(U1-GPIO7/SCL): track 56.8 -> 54.6 mm
